Commit message: updated automove and urdf

File: dingo_ws/src/dingo_description/urdf/dingo.urdf (robot description, URDF)
Before this commit: robot dingo, 17 links, 16 joints
Links:
- added link IMU_nose_frame, mass 0.002; collision box size=0.02 0.015 0.005; visual box size=0.02 0.015 0.005
- added link IMU_tail_frame, mass 0.002; collision box size=0.02 0.015 0.005; visual box size=0.02 0.015 0.005
- added link base_footprint
- added link laser_frame, mass 0.6; collision cylinder length=0.04 radius=0.05; visual cylinder length=0.04 radius=0.05
Joints:
- added joint IMU_nose_joint: type fixed, parent base_link, child IMU_nose_frame, origin xyz=0.18 0 0.04 rpy=0 0 0
- added joint IMU_tail_joint: type fixed, parent base_link, child IMU_tail_frame, origin xyz=-0.1685 0 0.04 rpy=0 0 0
- added joint base_footprint_joint: type fixed, parent base_link, child base_footprint, origin xyz=0 0 0 rpy=0 0 0
- added joint laser_joint: type fixed, parent base_link, child laser_frame, origin xyz=0.017 0 0.05 rpy=0 0 0

Commit message: got hector slam to work

File: dingo_ws/src/dingo_description/urdf/dingo.urdf (robot description, URDF)
Before this commit: robot dingo, 21 links, 20 joints
Links:
- removed link laser_frame
- added link laser, mass 0.6; collision cylinder length=0.04 radius=0.05; visual cylinder length=0.04 radius=0.05
Joints:
- joint laser_joint: child laser_frame -> laser
